Commit message: small changes

File: urdf/floating_base.urdf.xacro (robot description, xacro)
@@ -3,8 +3,6 @@
 <xacro:property name="PI" value="3.14159265359" />
 <xacro:property name="PI_2" value="1.57079632679" />
-<xacro:property name="print" value="true" />
 <xacro:macro name="floating_base_link" params="name">
 	<link name="floating_base_${name}">
-	<xacro:if value="${print}">
 	    <visual>
 	     <origin xyz="0 0 0" rpy="0 0 0" />
@@ -16,5 +14,4 @@
 	     </material>
 	   </visual>
-	</xacro:if>
 	</link>
 </xacro:macro>
@@ -25,7 +22,5 @@
           <origin xyz="0 0 0" rpy="0 0 0" />
           <axis xyz="${axis_xyz}" />
-          <xacro:if value="${print}">
-	    <limit velocity="1000.0" effort="1000.0" lower="-10.0" upper="10.0" />
-          </xacro:if>
+	  <limit velocity="1000.0" effort="1000.0" lower="-10.0" upper="10.0" />
         </joint>
 </xacro:macro>
